Commit message: working on spacecraft thruster force plugin

File: jksun_ws/src/spacecraft_simulator_description/urdf/spacecraft_simulator.urdf (robot description, URDF)
Before this commit: robot spacecraft_simulator, 1 links, 0 joints
Links:
- removed link base_link
- added link sc, mass 9.08; collision mesh filename=package://spacecraft_simulator_description/meshes/sc_simple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; visual mesh filename=package://spacecraft_simulator_description/meshes/sc_simple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
