Commit message: removing temp files

File: jksun_ws/src/spacecraft_simulator_description/urdf/3DOF_sc.urdf (robot description, URDF)
Before this commit: robot spacecraft_simulator, 1 links, 0 joints
Links:
- link sc: mass 9.08 -> 17.69

File: jksun_ws/src/spacecraft_simulator_description/urdf/5DOF_sc.urdf (robot description, URDF)
Before this commit: robot spacecraft_simulator, 1 links, 0 joints
Links:
- removed link sc
- added link base_link, mass 9.08; collision mesh filename=package://spacecraft_simulator_description/meshes/sc_simple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; visual mesh filename=package://spacecraft_simulator_description/meshes/sc_simple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
