Commit message: started 5DOF model

File: jksun_ws/src/spacecraft_simulator_description/urdf/5DOF_spacecraft_simulator.urdf (robot description, URDF)
Before this commit: robot spacecraft_simulator, 1 links, 0 joints
Links:
- added link upper_stage, mass 11.126; collision mesh filename=package://spacecraft_simulator_description/meshes/sc_top_ba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; visual mesh filename=package://spacecraft_simulator_description/meshes/sc_top_ba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
- link base_link: mass 9.08 -> 8.764; geometry collision mesh filename=package://spacecraft_simulator_description/meshes/sc_bot_ba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; visual mesh filename=package://spacecraft_simulator_description/meshes/sc_bot_ba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
Joints:
- added joint base_link_anchor: type revolute, parent upper_stage, child base_link, origin xyz=0 0 0.74522 rpy=0 0 0, axis 1 1 0, limit lower=-0.7854 upper=0.7854 effort=1000.0 velocity=0.5

Commit message: working on trajectory control

File: jksun_ws/src/spacecraft_simulator_description/urdf/5DOF_spacecraft_simulator.urdf (robot description, URDF)
Before this commit: robot spacecraft_simulator, 2 links, 1 joints
Joints:
- removed joint base_link_anchor
- added joint air_bearing: type revolute, parent base_link, child upper_stage, origin xyz=0 0 0 rpy=0 0 0, axis 1 1 0, limit lower=-0.7854 upper=0.7854 effort=1000.0 velocity=0.2
