Commit message: mostly completed 5-DOF model

File: jksun_ws/src/spacecraft_simulator_description/urdf/3DOF_spacecraft_simulator.urdf.xacro (robot description, xacro)
@@ -1,4 +1,7 @@
 <?xml version="1.0"?>
-<!-- Urdf format of the ARCL 3DOF spacecraft simulator. -->
+<!-- Xacro format of the ARCL 3DOF spacecraft simulator. Can be parsed into
+  an urdf. Xacro format used to pass in arguments for unique topic names for
+  each respective 3DOF spacecraft model.
+  Author: Jennifer Sun (jksun@caltech.edu) -->
 <robot name="spacecraft_simulator">
 <!--===========================================================================
@@ -6,5 +9,5 @@
 ============================================================================-->
   <!-- Represents the spacecraft simulator model -->
-  <link name="sc">
+  <link name="base_link">
     <inertial>
       <!-- Mass and inertia according to solidworks model of full 3DOF sc -->
@@ -24,5 +27,4 @@
     <visual>
       <geometry>
-        <!-- <mesh filename="package://spacecraft_simulator_description/meshes/spacecraft-simulator-simple.dae"/> -->
         <mesh filename="package://spacecraft_simulator_description/meshes/sc_simple_ball.dae"/>
       </geometry>
@@ -30,8 +32,7 @@
     <collision>
       <!-- Determines position on link where collision is checked -->
-      <origin xyz="0 0 0"/>
+      <origin xyz="0 0 0.41941"/>
       <geometry>
-        <mesh filename="package://spacecraft_simulator_description/meshes/sc_simple_ball_collision.dae"/>
-        <!-- <box>0.4572 0.4572 0.83882</box> -->
+        <box size="0.4572 0.4572 0.83882"/>
       </geometry>
       <surface>
@@ -56,23 +57,9 @@
 ============================================================================-->
   <gazebo>
-    <!-- Plugin that controls planar movement of the model using velocity. -->
-    <!-- <plugin name="object_controller" filename="libgazebo_ros_planar_move.so">
-      <commandTopic>cmd_vel</commandTopic>
-      <odometryTopic>odom</odometryTopic>
-      <odometryFrame>odom</odometryFrame>
-      <odometryRate>20.0</odometryRate>
-      <robotBaseFrame>sc</robotBaseFrame>
-    </plugin> -->
-    <!-- Plugin that controls movement of the model using forces and torques at
-    the model's center of mass. -->
-    <!-- <plugin name="force_controller" filename="libgazebo_ros_force.so">
-      <bodyName>sc</bodyName>
-      <topicName>ros_force</topicName>
-    </plugin> -->
     <!-- Plugin that controls movement of the model using forces at relative
     positions to the model's center of mass. Designed the model forces applied
     at specific thruster locations. -->
     <plugin name="thruster_force_controller" filename="libspacecraft_thruster8_force.so">
-      <bodyName>sc</bodyName>
+      <bodyName>base_link</bodyName>
       <topicName>$(arg spacecraft_name)/thruster8_force</topicName>
     </plugin>
@@ -83,5 +70,5 @@
       <alwaysOn>true</alwaysOn>
       <updateRate>100.0</updateRate>
-      <bodyName>sc</bodyName>
+      <bodyName>base_link</bodyName>
       <topicName>$(arg spacecraft_name)_pose</topicName>
       <gaussianNoise>0.0</gaussianNoise>
@@ -91,4 +78,18 @@
     </plugin>
   </gazebo>
+  <!-- Plugin that controls planar movement of the model using velocity. -->
+  <!-- <plugin name="object_controller" filename="libgazebo_ros_planar_move.so">
+    <commandTopic>cmd_vel</commandTopic>
+    <odometryTopic>odom</odometryTopic>
+    <odometryFrame>odom</odometryFrame>
+    <odometryRate>20.0</odometryRate>
+    <robotBaseFrame>base_link</robotBaseFrame>
+  </plugin> -->
+  <!-- Plugin that controls movement of the model using forces and torques at
+  the model's center of mass. -->
+  <!-- <plugin name="force_controller" filename="libgazebo_ros_force.so">
+    <bodyName>base_link</bodyName>
+    <topicName>ros_force</topicName>
+  </plugin> -->
   <!-- Specific format for gazebo sensor plugin. Uses a gazebo sensor for
   simulating an inertial mostion sensor. -->
@@ -102,5 +103,5 @@
       <plugin filename="libgazebo_ros_imu_sensor.so" name="imu_plugin">
         <topicName>$(arg spacecraft_name)/Imu</topicName>
-        <bodyName>sc</bodyName>
+        <bodyName>base_link</bodyName>
         <updateRateHZ>10.0</updateRateHZ>
         <gaussianNoise>0.0</gaussianNoise>

Commit message: testing w csv files

File: jksun_ws/src/spacecraft_simulator_description/urdf/3DOF_spacecraft_simulator.urdf.xacro (robot description, xacro)
@@ -11,15 +11,10 @@
   <link name="base_link">
     <inertial>
-      <!-- Mass and inertia according to solidworks model of full 3DOF sc -->
-      <!-- <mass value="9.08"/> -->
+      <!-- Mass according to rough measuring of the full 5DOF spacecraft -->
       <mass value="19.890"/>
       <!-- Sets up center of mass of link at the bottom of the ball joint -->
       <origin xyz="0 0 0.74522"/>
-      <!-- <inertia ixx="27.60" iyy="3.36" izz="28.06"
-               ixy="-5.21" ixz="0.86" iyz="-4.00"/> -->
-      <!-- From simplified 3DOF CAD -->
-      <!-- <inertia ixx="2.51" iyy="0.50" izz="2.60"
-               ixy="-0.55" ixz="0.16" iyz="-0.43"/> -->
-      <!-- From complete 5DOF CAD -->
+      <!-- Inertia according to solidworks model of the full 5DOF sc
+      upper stage -->
       <inertia ixx="4.09" iyy="0.68" izz="4.07"
                ixy="-0.11" ixz="0.03" iyz="-0.02"/>

File: jksun_ws/src/spacecraft_simulator_description/urdf/5DOF_spacecraft_simulator.urdf.xacro (robot description, xacro)
@@ -1,5 +1,11 @@
 <?xml version="1.0"?>
-<!-- Urdf format of the ARCL 5DOF spacecraft simulator. -->
+<!-- Xacro format of the ARCL 5DOF spacecraft simulator. Can be parsed into
+  an urdf. Xacro format used to pass in arguments for unique topic names for
+  each respective 5DOF spacecraft model.
+  Author: Jennifer Sun (jksun@caltech.edu) -->
 <robot name="spacecraft_simulator">
+<!--===========================================================================
+SPACECRAFT SIMULATOR MODEL (specifies urdf link properties for 3DOF sc model)
+============================================================================-->
   <!-- Represents a simplified pedestal design for the spacecraft simulator
   model -->
@@ -33,5 +39,4 @@
       <origin xyz="0 0 0.02521"/>
       <geometry>
-        <!-- <mesh filename="package://spacecraft_simulator_description/meshes/sc_bot_ball_v2.dae"/> -->
         <cylinder radius="0.2159" length="0.05042"/>
       </geometry>
@@ -145,4 +150,7 @@
     </collision>
   </link>
+<!--===========================================================================
+GAZEBO PLUGINS (plugins used to connect ROS with the Gazebo model)
+============================================================================-->
   <gazebo>
     <!-- Plugin that controls movement of the model using forces at relative
@@ -153,4 +161,7 @@
       <topicName>$(arg spacecraft_name)/thruster16_force</topicName>
     </plugin>
+    <!-- Plugin that provides a 3D position interface for ground truth.
+    Publishes pose of the spacecraft link in simulation using Odometry
+    messages. -->
     <plugin name="sc_model_pose" filename="libgazebo_ros_p3d.so">
       <alwaysOn>true</alwaysOn>
